File: Schematic/ButtonBox.kicad_pcb (KiCad board)
At the start: 2 copper layers, 56.4 x 42.7 mm, 15 parts, among them P1 JOY_THRUST, P10 SW_CARGO, P2 JOY_NAVI, P3 SW_FSHIFT, P4 SW_SILENT, P5 SW_DUMP, P6 SW_DEPLOY, P7 SW_LIGHTS, P8 SW_LANDING, P9 SW_FUEL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

Commit message: Single board design.
Parts:
- P1, P2: footprint Pin_Headers:Pin_Header_Angled_1x05 -> Pin_Headers:Pin_Header_Straight_1x05
- P10, P3, P4, P5, P6, P7, P8, P9: footprint Pin_Headers:Pin_Header_Angled_1x02 -> Pin_Headers:Pin_Header_Straight_1x02
Routing:
- net /clockEn: track 45.5 -> 41.7 mm
- net VCC: track 178.4 -> 176.4 mm
- net /SW_LIGHTS: track 33.5 -> 34.6 mm
- net /SW_DUMP: track 22.5 -> 23.4 mm
- net /SW_SILENT: track 20.4 -> 21.2 mm
